Commit message: Fase 2: Pepper en Gazebo Harmonic con los controladores del V8
- pepper_control: controladores con los nombres del V8 (LeftArm_controller,
  RightArm_controller, Head_controller, Pelvis_controller, manos y
  joint_state_controller = JointStateBroadcaster), topic ~/command conservado
  con un remapeo, y launch de rqt_joint_trajectory_controller con remapeos.
- pepper_gazebo_plugin: launch para el mundo vacío (spawn como pepper_MP),
  mundo SDF y arms_down.sh portado a ROS 2.
- pepper_description: bloque ros2_control para gz_ros2_control, hook de
  GZ_SIM_RESOURCE_PATH, masa de los grippers corregida (DART abortaba) y
  posición inicial válida para LHand/RHand.
- README: sección de la Fase 2, tabla de nomenclatura ampliada y capturas.

Co-Authored-By: Claude Opus 5.5 (1M context) <noreply@anthropic.com>

File: pepper_description/urdf/pepper_arms.xacro (robot description, xacro)
@@ -88,6 +88,8 @@
 	<link name="l_gripper">
 		<inertial>
-			<mass value="2e-06"/>
-			<inertia ixx="1.1e-09" ixy="0" ixz="0" iyy="1.1e-09" iyz="0" izz="1.1e-09"/>
+			<!-- V9: el V8 tenía 2e-06 kg / 1.1e-09; DART (Gazebo Harmonic) aborta con cuerpos tan
+			     ligeros colgando de un joint revolute. Masa aproximada de la mano. -->
+			<mass value="0.05"/>
+			<inertia ixx="1e-05" ixy="0" ixz="0" iyy="1e-05" iyz="0" izz="1e-05"/>
 		</inertial>
 	</link>
@@ -176,6 +178,8 @@
 	<link name="r_gripper">
 		<inertial>
-			<mass value="2e-06"/>
-			<inertia ixx="1.1e-09" ixy="0" ixz="0" iyy="1.1e-09" iyz="0" izz="1.1e-09"/>
+			<!-- V9: el V8 tenía 2e-06 kg / 1.1e-09; DART (Gazebo Harmonic) aborta con cuerpos tan
+			     ligeros colgando de un joint revolute. Masa aproximada de la mano. -->
+			<mass value="0.05"/>
+			<inertia ixx="1e-05" ixy="0" ixz="0" iyy="1e-05" iyz="0" izz="1e-05"/>
 		</inertial>
 	</link>

File: pepper_description/urdf/pepper_robot.urdf.xacro (robot description, xacro)
@@ -5,4 +5,7 @@
   <!-- Dedos: el V8 los deja fuera en simulación (pepper_robot_CPU.xacro) -->
   <xacro:arg name="fingers" default="false"/>
+  <!-- Gazebo Harmonic: añade ros2_control (lo pasa pepper_gazebo_plugin) -->
+  <xacro:arg name="gazebo" default="false"/>
+  <xacro:arg name="controllers_file" default=""/>
   <xacro:include filename="$(find pepper_description)/urdf/pepper_visual_collisions.xacro"/>
   <xacro:include filename="$(find pepper_description)/urdf/pepper_head.xacro"/>
@@ -15,3 +18,7 @@
     <xacro:include filename="$(find pepper_description)/urdf/pepper_fingers.xacro"/>
   </xacro:if>
+  <xacro:if value="$(arg gazebo)">
+    <xacro:include filename="$(find pepper_description)/urdf/pepper_ros2_control.xacro"/>
+    <xacro:pepper_ros2_control controllers_file="$(arg controllers_file)"/>
+  </xacro:if>
 </robot>
