Commit message: Fase 4: sensores de Pepper con los topics y frames del V8
- pepper_sensors_gazebo.xacro: cámaras front/bottom, rgbd (depth + ir),
  3 láseres, hokuyo falso y sonares, con los parámetros del V8 y gz_frame_id.
- pepper_bridge.yaml: ros_gz_bridge con los nombres del V8.
- laser_publisher.py (port del V8) para /pepper/laser_2 y /cloud*;
  sonar_to_range (C++) para /pepper/sonar_*; depth_image_proc para
  /pepper/camera/depth/points en el frame óptico.
- Ruedas en ros2_control solo con estado: sus TF existen (arregla el error
  de RViz que el V8 esquivaba comentando líneas).
- pepper_sensors.rviz para RViz2 y su launch.
- README: Fase 4 con topics, verificación y cambios respecto al V8.

Co-Authored-By: Claude Opus 5.5 (1M context) <noreply@anthropic.com>

File: pepper_description/urdf/pepper_robot.urdf.xacro (robot description, xacro)
@@ -22,4 +22,5 @@
     <xacro:pepper_ros2_control controllers_file="$(arg controllers_file)"/>
     <xacro:include filename="$(find pepper_description)/urdf/pepper_gazebo.xacro"/>
+    <xacro:include filename="$(find pepper_description)/urdf/pepper_sensors_gazebo.xacro"/>
   </xacro:if>
 </robot>

File: pepper_description/urdf/pepper_ros2_control.xacro (robot description, xacro)
@@ -1,6 +1,7 @@
 <?xml version="1.0"?>
 <!-- ros2_control para Gazebo Harmonic. Sustituye a pepperGazebo*.xacro (gazebo_ros_control)
-     y pepperTransmission*.xacro del V8. Las ruedas no van aquí: la base se mueve con su
-     propio plugin (Fase 3), como en el V8. -->
+     y pepperTransmission*.xacro del V8. Las ruedas sólo tienen interfaces de estado: la base
+     se mueve con su propio plugin (Fase 3), como en el V8, pero así joint_state_controller
+     publica WheelB/FL/FR y existen sus TF (en el V8 había que comentarlas para RViz). -->
 <robot xmlns:xacro="http://www.ros.org/wiki/xacro">
   <xacro:macro name="pepper_joint" params="name initial:=0.0">
@@ -39,4 +40,17 @@
       <xacro:pepper_joint name="RWristYaw"/>
       <xacro:pepper_joint name="RHand" initial="0.5"/>
+      <!-- Ruedas: sólo estado -->
+      <joint name="WheelB">
+        <state_interface name="position"/>
+        <state_interface name="velocity"/>
+      </joint>
+      <joint name="WheelFL">
+        <state_interface name="position"/>
+        <state_interface name="velocity"/>
+      </joint>
+      <joint name="WheelFR">
+        <state_interface name="position"/>
+        <state_interface name="velocity"/>
+      </joint>
     </ros2_control>
     <gazebo>
